Commit message: inertial property

File: src/abb_irb6640_support/urdf/irb6640_185_280_macro.xacro (robot description, xacro)
@@ -18,5 +18,5 @@
       </visual>
       <inertial>
-        <mass value="1"/>
+        <mass value="500"/>
         <inertia ixx="1.0" ixy="1.0" ixz="1.0" iyy="1.0" iyz="1.0" izz="1.0" />
       </inertial>
@@ -35,6 +35,6 @@
       </visual>
       <inertial>
-        <mass value="1"/>
-        <inertia ixx="1.0" ixy="1.0" ixz="1.0" iyy="1.0" iyz="1.0" izz="1.0" />
+        <mass value="411"/>
+        <inertia ixx="0.1315" ixy="0.001" ixz="0.001" iyy="0.1415" iyz="0.001" izz="0.02" />
       </inertial>
     </link>
@@ -52,6 +52,6 @@
       </visual>
       <inertial>
-        <mass value="1"/>
-        <inertia ixx="1.0" ixy="1.0" ixz="1.0" iyy="1.0" iyz="1.0" izz="1.0" />
+        <mass value="121"/>
+        <inertia ixx="0.02" ixy="0.001" ixz="0.001" iyy="0.3962" iyz="0.001" izz="0.3952" />
       </inertial>
     </link>
@@ -69,6 +69,6 @@
       </visual>
       <inertial>
-        <mass value="1"/>
-        <inertia ixx="1.0" ixy="1.0" ixz="1.0" iyy="1.0" iyz="1.0" izz="1.0" />
+        <mass value="113.4"/>
+        <inertia ixx="0.045" ixy="0.001" ixz="0.001" iyy="0.04" iyz="0.001" izz="0.012" />
       </inertial>
     </link>
@@ -86,6 +86,6 @@
       </visual>
       <inertial>
-        <mass value="1"/>
-        <inertia ixx="1.0" ixy="1.0" ixz="1.0" iyy="1.0" iyz="1.0" izz="1.0" />
+        <mass value="74.6"/>
+        <inertia ixx="0.437" ixy="0.001" ixz="0.001" iyy="0.447" iyz="0.001" izz="0.02" />
       </inertial>
     </link>
@@ -103,6 +103,6 @@
       </visual>
       <inertial>
-        <mass value="1"/>
-        <inertia ixx="1.0" ixy="1.0" ixz="1.0" iyy="1.0" iyz="1.0" izz="1.0" />
+        <mass value="24.6"/>
+        <inertia ixx="0.0133" ixy="0.001" ixz="0.001" iyy="0.025" iyz="0.001" izz="0.02" />
       </inertial>
     </link>
@@ -120,6 +120,6 @@
       </visual>
       <inertial>
-        <mass value="1"/>
-        <inertia ixx="1.0" ixy="1.0" ixz="1.0" iyy="1.0" iyz="1.0" izz="1.0" />
+        <mass value="5"/>
+        <inertia ixx="0.02" ixy="0.001" ixz="0.001" iyy="0.02" iyz="0.001" izz="0.02" />
       </inertial>
     </link>
@@ -139,5 +139,5 @@
       </visual>
       <inertial>
-        <mass value="1"/>
+        <mass value="200"/>
         <inertia ixx="1.0" ixy="1.0" ixz="1.0" iyy="1.0" iyz="1.0" izz="1.0" />
       </inertial>
@@ -156,5 +156,5 @@
       </visual>
       <inertial>
-        <mass value="1"/>
+        <mass value="10"/>
         <inertia ixx="1.0" ixy="1.0" ixz="1.0" iyy="1.0" iyz="1.0" izz="1.0" />
       </inertial>
