Commit message: add

File: src/abb_irb6640_gazebo/urdf/irb6640_185_280.xacro (robot description, xacro)
@@ -5,7 +5,23 @@
   <!-- connect robot with world -->
   <link name="world" />
-  <joint name="world_to_base_link_joint" type="fixed">
+  <link name="workcell">
+    <visual>
+      <origin xyz="-1.256 -2.635 0" rpy="0 0 0" />
+      <geometry>
+        <mesh filename="package://abb_irb6640_support/meshes/irb6640_185_280/visual/workcell.STL" scale="0.001 0.001 0.001" />
+      </geometry>
+    </visual>
+    <inertial>
+      <mass value="92.5052"/>
+      <inertia ixx="1.0" ixy="1.0" ixz="1.0" iyy="1.0" iyz="1.0" izz="1.0" />
+    </inertial>
+  </link>
+  <joint name="world_to_base" type="fixed">
     <parent link="world" />
     <child link="base_link" />
+  </joint>
+  <joint name="workcell" type="fixed">
+    <parent link="world" />
+    <child link="workcell" />
   </joint>
   <!-- ros_control plugin -->

File: src/abb_irb6640_gazebo/urdf/irb6640_185_280_macro.xacro (robot description, xacro)
@@ -66,10 +66,4 @@
       </actuator>
     </transmission>
-    <gazebo>
-     <plugin name="joint_state_publisher"
-          filename="libgazebo_ros_joint_state_publisher.so">
-      <jointName>joint_1, joint_2, joint_3, joint_4, joint_5, joint_6</jointName>
-    </plugin>
-    </gazebo>
     <!-- end of transmission list -->
     <!-- Gazebo-specific link properties -->

File: src/abb_irb6640_support/urdf/irb6640_185_280.urdf (robot description, URDF)
Before this commit: robot abb_irb6640_185_280, 11 links, 10 joints
Links:
- link base_link: mass None -> 500
- link link_1: mass None -> 411
- link link_2: mass None -> 121
- link link_3: mass None -> 113.4
- link link_4: mass None -> 74.6
- link link_5: mass None -> 24.6
- link link_6: mass None -> 5
- link link_cylinder: mass None -> 200
- link link_piston: mass None -> 10
Joints:
- joint joint_1: limit lower=-2.967 upper=2.967 effort=0 velocity=1.7453 -> lower=-2.967 upper=2.967 effort=1000 velocity=1.7453
- joint joint_2: limit lower=-1.134 upper=1.4855 effort=0 velocity=1.5707 -> lower=-1.134 upper=1.4855 effort=1000 velocity=1.5707
- joint joint_3: limit lower=-3.142 upper=1.222 effort=0 velocity=1.5707 -> lower=-3.142 upper=1.222 effort=1000 velocity=1.5707
- joint joint_4: limit lower=-5.236 upper=5.236 effort=0 velocity=2.9671 -> lower=-5.236 upper=5.236 effort=1000 velocity=2.9671
- joint joint_5: limit lower=-2.094 upper=2.094 effort=0 velocity=2.4435 -> lower=-2.094 upper=2.094 effort=1000 velocity=2.4435
- joint joint_6: limit lower=-6.283 upper=6.283 effort=0 velocity=3.3161 -> lower=-6.283 upper=6.283 effort=1000 velocity=3.3161

File: src/abb_irb6640_support/urdf/irb6640_185_280_macro.xacro (robot description, xacro)
@@ -10,4 +10,5 @@
       </collision>
       <visual name="visual">
+        <origin xyz="0 0 0.05" rpy="0 0 0" />
         <geometry>
           <mesh filename="package://abb_irb6640_support/meshes/irb6640_185_280/visual/base_link.dae"/>
@@ -18,5 +19,5 @@
       </visual>
       <inertial>
-        <mass value="500"/>
+        <mass value="1"/>
         <inertia ixx="1.0" ixy="1.0" ixz="1.0" iyy="1.0" iyz="1.0" izz="1.0" />
       </inertial>
@@ -35,6 +36,6 @@
       </visual>
       <inertial>
-        <mass value="411"/>
-        <inertia ixx="0.1315" ixy="0.001" ixz="0.001" iyy="0.1415" iyz="0.001" izz="0.02" />
+        <mass value="1"/>
+        <inertia ixx="1.0" ixy="1.0" ixz="1.0" iyy="1.0" iyz="1.0" izz="1.0" />
       </inertial>
     </link>
@@ -52,6 +53,6 @@
       </visual>
       <inertial>
-        <mass value="121"/>
-        <inertia ixx="0.02" ixy="0.001" ixz="0.001" iyy="0.3962" iyz="0.001" izz="0.3952" />
+        <mass value="1"/>
+        <inertia ixx="1.0" ixy="1.0" ixz="1.0" iyy="1.0" iyz="1.0" izz="1.0" />
       </inertial>
     </link>
@@ -69,6 +70,6 @@
       </visual>
       <inertial>
-        <mass value="113.4"/>
-        <inertia ixx="0.045" ixy="0.001" ixz="0.001" iyy="0.04" iyz="0.001" izz="0.012" />
+        <mass value="1"/>
+        <inertia ixx="1.0" ixy="1.0" ixz="1.0" iyy="1.0" iyz="1.0" izz="1.0" />
       </inertial>
     </link>
@@ -86,6 +87,6 @@
       </visual>
       <inertial>
-        <mass value="74.6"/>
-        <inertia ixx="0.437" ixy="0.001" ixz="0.001" iyy="0.447" iyz="0.001" izz="0.02" />
+        <mass value="1"/>
+        <inertia ixx="1.0" ixy="1.0" ixz="1.0" iyy="1.0" iyz="1.0" izz="1.0" />
       </inertial>
     </link>
@@ -103,6 +104,6 @@
       </visual>
       <inertial>
-        <mass value="24.6"/>
-        <inertia ixx="0.0133" ixy="0.001" ixz="0.001" iyy="0.025" iyz="0.001" izz="0.02" />
+        <mass value="1"/>
+        <inertia ixx="1.0" ixy="1.0" ixz="1.0" iyy="1.0" iyz="1.0" izz="1.0" />
       </inertial>
     </link>
@@ -120,6 +121,6 @@
       </visual>
       <inertial>
-        <mass value="5"/>
-        <inertia ixx="0.02" ixy="0.001" ixz="0.001" iyy="0.02" iyz="0.001" izz="0.02" />
+        <mass value="1"/>
+        <inertia ixx="1.0" ixy="1.0" ixz="1.0" iyy="1.0" iyz="1.0" izz="1.0" />
       </inertial>
     </link>
@@ -139,5 +140,5 @@
       </visual>
       <inertial>
-        <mass value="200"/>
+        <mass value="1"/>
         <inertia ixx="1.0" ixy="1.0" ixz="1.0" iyy="1.0" iyz="1.0" izz="1.0" />
       </inertial>
@@ -156,5 +157,5 @@
       </visual>
       <inertial>
-        <mass value="10"/>
+        <mass value="1"/>
         <inertia ixx="1.0" ixy="1.0" ixz="1.0" iyy="1.0" iyz="1.0" izz="1.0" />
       </inertial>

Commit message: opencv

File: src/abb_irb6640_gazebo/urdf/irb6640_185_280.xacro (robot description, xacro)
@@ -2,4 +2,9 @@
 <robot name="abb_irb6640_185_280" xmlns:xacro="http://ros.org/wiki/xacro">
   <xacro:include filename="$(find abb_irb6640_gazebo)/urdf/irb6640_185_280_macro.xacro" />
+  <xacro:include filename="$(find abb_irb6640_gazebo)/urdf/sensors/xtion_pro_live.urdf.xacro"/>
+  <xacro:property name="deg_to_rad" value="0.01745329251994329577"/>
+  <!-- Constants -->
+  <xacro:property name="M_SCALE" value="0.001 0.001 0.001"/>
+  <xacro:property name="M_PI" value="3.14159"/>
   <xacro:abb_irb6640_185_280_gazebo prefix="" />
   <!-- connect robot with world -->
@@ -25,4 +30,9 @@
     <child link="workcell" />
   </joint>
+    <!-- Define RGB-D sensor -->
+  <xacro:xtion_pro_live name="rgbd_camera" parent="base">
+    <origin xyz="3.07 -1.6 2.4" rpy="0 ${75.0 * deg_to_rad} 0"/>
+    <origin xyz="0 0 0" rpy="${-90.0 * deg_to_rad} 0 ${-90.0 * deg_to_rad}"/>
+  </xacro:xtion_pro_live>
   <!-- ros_control plugin -->
   <gazebo>
